File: Pikachuu40-ProMicro/Pikachuu40-ProMicro.kicad_pcb (KiCad board)
At the start: 2 copper layers, 93 parts, among them K1 KEYSW, K10 KEYSW, K11 KEYSW, K12 KEYSW, K13 KEYSW, K14 KEYSW, K15 KEYSW, K16 KEYSW, K17 KEYSW, K18 KEYSW, K19 KEYSW, K2 KEYSW, K20 KEYSW, K21 KEYSW, K22 KEYSW, K23 KEYSW, K24 KEYSW, K25 KEYSW, K26 KEYSW, K27 KEYSW, K28 KEYSW, K29 KEYSW, K3 KEYSW, K30 KEYSW, K31 KEYSW, K32 KEYSW, K33 KEYSW, K34 KEYSW, K35 KEYSW, K36 KEYSW, K37 KEYSW, K38 KEYSW, K39 KEYSW, K4 KEYSW, K40 KEYSW, K41 KEYSW, K42 KEYSW, K43 KEYSW, K44 KEYSW, K45 KEYSW, K5 KEYSW, K6 KEYSW, K7 KEYSW, K8 KEYSW, K9 KEYSW, U1 ProMicro

Commit message: Rough Routing Done
Parts:
- removed D46: D, Keebio-Parts:Diode
- removed K?1: KEYSW, Button_Switch_Keyboard:SW_Cherry_MX_1.00u_PCB
- D1, D10, D11, D12, D13, D14, D15, D16, D17, D18, D19, D2, D20, D21, D22, D23, D24, D25, D26, D27, D28, D29, D3, D30, D31, D32, D33, D34, D35, D36, D37, D38, D39, D4, D40, D41, D42, D43, D44, D45, D5, D6, D7, D8, D9: moved to B.Cu
- moved K39 710.6 mm to (310.3, 101.0)
- moved K37 698.9 mm to (272.2, 101.0)
- moved D39 684.4 mm to (299.6, 107.3), turned to 90 degrees
- moved K38 681.0 mm to (291.2, 101.0)
- moved K45 672.2 mm to (253.1, 120.0)
- moved K36 659.0 mm to (253.1, 101.0)
- moved D38 656.7 mm to (280.4, 107.3), turned to 90 degrees
- moved D45 647.5 mm to (242.4, 126.4), turned to 90 degrees
- moved D37 647.3 mm to (261.4, 107.3), turned to 90 degrees
- moved K24 645.3 mm to (272.2, 81.9)
- moved D25 645.0 mm to (287.4, 88.3), turned to 90 degrees
- moved K44 632.9 mm to (231.5, 120.0)
- moved D35 632.3 mm to (223.0, 107.3), turned to 90 degrees
- moved D44 626.0 mm to (220.6, 126.4), turned to 90 degrees
- moved D12 622.4 mm to (270.9, 69.2), turned to 90 degrees
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Connections:
- D10 pad 1: ROW4 -> ROW0
- D12 pad 1: ROW1 -> ROW0
- D13 pad 1: ROW2 -> ROW1
- D14 pad 1: ROW3 -> ROW1
- D15 pad 1: ROW0 -> ROW1
- D17 pad 1: ROW2 -> ROW1
- D18 pad 1: ROW3 -> ROW1
- D19 pad 1: ROW0 -> ROW1
- D2 pad 1: ROW1 -> ROW0
- D2 pad 2: ROW0 -> Net-(D2-Pad2)
- D21 pad 1: ROW2 -> ROW1
- D22 pad 1: ROW3 -> ROW1
- D23 pad 1: ROW0 -> ROW1
- D25 pad 1: ROW2 -> ROW1
- D26 pad 1: ROW3 -> ROW2
- D27 pad 1: ROW0 -> ROW2
- D28 pad 1: ROW1 -> ROW2
- D3 pad 1: ROW2 -> ROW0
- D3 pad 2: ROW1 -> Net-(D3-Pad2)
- D30 pad 1: ROW3 -> ROW2
- D31 pad 1: ROW0 -> ROW2
- D32 pad 1: ROW1 -> ROW2
- D34 pad 1: ROW3 -> ROW2
- D35 pad 1: ROW0 -> ROW2
- D36 pad 1: ROW1 -> ROW2
- D38 pad 1: ROW3 -> ROW2
- D39 pad 1: ROW0 -> ROW2
- D4 pad 1: ROW3 -> ROW0
- D4 pad 2: ROW2 -> Net-(D4-Pad2)
- D40 pad 1: ROW1 -> ROW3
- D41 pad 1: ROW2 -> ROW3
- D43 pad 1: ROW0 -> ROW3
- D44 pad 1: ROW1 -> ROW3
- D45 pad 1: ROW2 -> ROW3
- D5 pad 1: ROW4 -> ROW0
- D5 pad 2: ROW3 -> Net-(D5-Pad2)
- D7 pad 1: ROW1 -> ROW0
- D8 pad 1: ROW2 -> ROW0
- D9 pad 1: ROW3 -> ROW0
- K1 pad 2: ROW0 -> Net-(D1-Pad2)
- K10 pad 1: COL2 -> COL9
- K10 pad 2: Net-(D11-Pad2) -> Net-(D10-Pad2)
- K11 pad 1: COL2 -> COLA
- K11 pad 2: Net-(D12-Pad2) -> Net-(D11-Pad2)
- K12 pad 1: COL2 -> COLB
- K12 pad 2: Net-(D13-Pad2) -> Net-(D12-Pad2)
- K13 pad 1: COL2 -> COL0
- K13 pad 2: Net-(D14-Pad2) -> Net-(D13-Pad2)
- K14 pad 1: COL3 -> COL1
- K14 pad 2: Net-(D15-Pad2) -> Net-(D14-Pad2)
- K15 pad 1: COL3 -> COL2
- K15 pad 2: Net-(D16-Pad2) -> Net-(D15-Pad2)
- K16 pad 2: Net-(D17-Pad2) -> Net-(D16-Pad2)
- K17 pad 1: COL3 -> COL4
- K17 pad 2: Net-(D18-Pad2) -> Net-(D17-Pad2)
- K18 pad 1: COL4 -> COL5
- K18 pad 2: Net-(D19-Pad2) -> Net-(D18-Pad2)
- K19 pad 1: COL4 -> COL6
- K19 pad 2: Net-(D20-Pad2) -> Net-(D19-Pad2)
- K2 pad 1: COL0 -> COL1
- K2 pad 2: ROW1 -> Net-(D2-Pad2)
- K20 pad 1: COL4 -> COL7
- K20 pad 2: Net-(D21-Pad2) -> Net-(D20-Pad2)
- K21 pad 1: COL4 -> COL8
- K21 pad 2: Net-(D22-Pad2) -> Net-(D21-Pad2)
- K22 pad 1: COL5 -> COL9
- K22 pad 2: Net-(D23-Pad2) -> Net-(D22-Pad2)
- K23 pad 1: COL5 -> COLA
- K23 pad 2: Net-(D24-Pad2) -> Net-(D23-Pad2)
- K24 pad 1: COL5 -> COLB
- K24 pad 2: Net-(D25-Pad2) -> Net-(D24-Pad2)
- K25 pad 1: COL5 -> COLB
- K25 pad 2: Net-(D26-Pad2) -> Net-(D25-Pad2)
- K26 pad 1: COL6 -> COL0
- K26 pad 2: Net-(D27-Pad2) -> Net-(D26-Pad2)
- K27 pad 1: COL6 -> COL1
- K27 pad 2: Net-(D28-Pad2) -> Net-(D27-Pad2)
- K28 pad 1: COL6 -> COL2
- K28 pad 2: Net-(D29-Pad2) -> Net-(D28-Pad2)
- K29 pad 1: COL6 -> COL3
- K29 pad 2: Net-(D30-Pad2) -> Net-(D29-Pad2)
- K3 pad 1: COL0 -> COL2
- K3 pad 2: ROW2 -> Net-(D3-Pad2)
- K30 pad 1: COL7 -> COL4
- K30 pad 2: Net-(D31-Pad2) -> Net-(D30-Pad2)
- K31 pad 1: COL7 -> COL5
- K31 pad 2: Net-(D32-Pad2) -> Net-(D31-Pad2)
- K32 pad 1: COL7 -> COL6
- K32 pad 2: Net-(D33-Pad2) -> Net-(D32-Pad2)
- K33 pad 2: Net-(D34-Pad2) -> Net-(D33-Pad2)
- K34 pad 2: Net-(D35-Pad2) -> Net-(D34-Pad2)
- K35 pad 1: COL8 -> COL9
- K35 pad 2: Net-(D36-Pad2) -> Net-(D35-Pad2)
- K36 pad 1: COL8 -> COLA
- K36 pad 2: Net-(D37-Pad2) -> Net-(D36-Pad2)
- K37 pad 1: COL8 -> COLB
- K37 pad 2: Net-(D38-Pad2) -> Net-(D37-Pad2)
- K38 pad 1: COL9 -> COLB
- K38 pad 2: Net-(D39-Pad2) -> Net-(D38-Pad2)
- K39 pad 1: COL9 -> COLB
- K39 pad 2: Net-(D40-Pad2) -> Net-(D39-Pad2)
- K4 pad 1: COL0 -> COL3
- K4 pad 2: ROW3 -> Net-(D4-Pad2)
- K40 pad 1: COL9 -> COL1
- K40 pad 2: Net-(D41-Pad2) -> Net-(D40-Pad2)
- K41 pad 1: COL9 -> COL2
- K41 pad 2: Net-(D42-Pad2) -> Net-(D41-Pad2)
- K42 pad 1: COL10 -> COL4
- K42 pad 2: Net-(D43-Pad2) -> Net-(D42-Pad2)
- K43 pad 1: COL10 -> COL7
- K43 pad 2: Net-(D44-Pad2) -> Net-(D43-Pad2)
- K44 pad 1: COL10 -> COL9
- K44 pad 2: Net-(D45-Pad2) -> Net-(D44-Pad2)
- K45 pad 1: COL10 -> COLA
- K45 pad 2: Net-(D46-Pad2) -> Net-(D45-Pad2)
- K5 pad 1: COL1 -> COL4
- K5 pad 2: Net-(D6-Pad2) -> Net-(D5-Pad2)
- K6 pad 1: COL1 -> COL5
- K6 pad 2: Net-(D7-Pad2) -> Net-(D6-Pad2)
- K7 pad 1: COL1 -> COL6
- K7 pad 2: Net-(D8-Pad2) -> Net-(D7-Pad2)
- K8 pad 1: COL1 -> COL7
- K8 pad 2: Net-(D9-Pad2) -> Net-(D8-Pad2)
- K9 pad 1: COL1 -> COL8
- K9 pad 2: Net-(D10-Pad2) -> Net-(D9-Pad2)
- U1 pad 11: COL6 -> ROW0
- U1 pad 12: COL7 -> ROW3
- U1 pad 13: COL8 -> ROW2
- U1 pad 14: COL9 -> ROW1
- U1 pad 15: COL10 -> COL6
- U1 pad 16: ROW0 -> COL7
- U1 pad 17: ROW1 -> COL8
- U1 pad 18: ROW2 -> COL9
- U1 pad 19: ROW3 -> COLA
- U1 pad 20: ROW4 -> COLB
Routing:
- net ROW2: track 0.00 -> 659.9 mm
- net ROW3: track 0.00 -> 518.6 mm
- net ROW1: track 0.00 -> 316.8 mm
- net ROW0: track 0.00 -> 297.9 mm
- net COLB: track 0.00 -> 260.8 mm
- net COL1: track 0.00 -> 190.1 mm
- net COL0: track 0.00 -> 188.1 mm
- net COLA: track 0.00 -> 176.9 mm
- net COL2: track 0.00 -> 172.3 mm
- net COL9: track 0.00 -> 159.4 mm
- net COL4: track 0.00 -> 135.0 mm
- net COL3: track 0.00 -> 130.6 mm
- net COL7: track 0.00 -> 121.8 mm
- net COL8: track 0.00 -> 121.7 mm
- net COL5: track 0.00 -> 94.6 mm
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Other:
- board outline added: 355.7 x 88.5 mm
- board text added: "I don't know what I'm doing to be honest"
- board text added: "Pro Micro"
